File: hardware/ultraflat.kicad_sch (KiCad schematic)
At the start: 91 parts, among them J1 USB_C_Receptacle_USB2.0_14P, SW1 SW_Push, SW10 SW_Push, SW11 SW_Push, SW12 SW_Push, SW13 SW_Push, SW14 SW_Push, SW15 SW_Push, SW16 SW_Push, SW17 SW_Push, SW18 SW_Push, SW19 SW_Push, SW2 SW_Push, SW20 SW_Push, SW21 SW_Push, SW22 SW_Push, SW23 SW_Push, SW24 SW_Push, SW25 SW_Push, SW26 SW_Push, SW27 SW_Push, SW28 SW_Push, SW29 SW_Push, SW3 SW_Push, SW30 SW_Push, SW4 SW_Push, SW5 SW_Push, SW6 SW_Push, SW7 SW_Push, SW8 SW_Push, SW9 SW_Push, U1 nRF52840, Y1 32MHz, Y2 32.768kHz

Commit message: Finish most of schem
Parts:
- added C21, C22: 4.7uF, Capacitor_SMD:C_0603_1608Metric, symbol Device:C
- added D31: LED, symbol Device:LED
- added J2: Conn_01x02, Connector_PinSocket_2.54mm:PinSocket_1x02_P2.54mm_Vertical, symbol Connector_Generic:Conn_01x02
- added J3: USB_C_Receptacle_USB2.0_14P, Connector_USB:USB_C_Receptacle_HRO_TYPE-C-31-M-12, symbol Connector:USB_C_Receptacle_USB2.0_14P
- added JP1: SolderJumper_2_Open, Jumper:SolderJumper-2_P1.3mm_Open_RoundedPad1.0x1.5mm, symbol Jumper:SolderJumper_2_Open
- added Q2: 2N7002, Package_TO_SOT_SMD:SOT-23, symbol Transistor_FET:2N7002
- added R10, R3, R6, R8: 10k, Resistor_SMD:R_0402_1005Metric_Pad0.72x0.64mm_HandSolder, symbol Device:R
- added R11, R12: 5.1k, Resistor_SMD:R_0402_1005Metric_Pad0.72x0.64mm_HandSolder, symbol Device:R
- added R4: 3.9k, Resistor_SMD:R_0402_1005Metric_Pad0.72x0.64mm_HandSolder, symbol Device:R
- added R5, R9: 1.5k, Resistor_SMD:R_0402_1005Metric_Pad0.72x0.64mm_HandSolder, symbol Device:R
- added R7: 100, Resistor_SMD:R_0402_1005Metric_Pad0.72x0.64mm_HandSolder, symbol Device:R
- added SW31: SW_SPDT, symbol Switch:SW_SPDT
- added U2: BQ24075RGT, Package_DFN_QFN:VQFN-16-1EP_3x3mm_P0.5mm_EP1.6x1.6mm, symbol Battery_Management:BQ24075RGT
- AE1: now left out of the parts list
- C1, C2, C3, C4: value C_Small -> 15pF; footprint (none) -> Capacitor_SMD:C_0402_1005Metric
- J1: footprint (none) -> Connector_USB:USB_C_Receptacle_HRO_TYPE-C-31-M-12; LCSC Part # (none) -> C165948
- R1, R2: footprint (none) -> Resistor_SMD:R_0402_1005Metric_Pad0.72x0.64mm_HandSolder
- SW1, SW10, SW11, SW12, SW13, SW14, SW15, SW16, SW17, SW18, SW19, SW2, SW20, SW21, SW22, SW23, SW24, SW25, SW26, SW27, SW28, SW29, SW3, SW30, SW4, SW5, SW6, SW7, SW8, SW9: symbol Switch:SW_Push -> ultraflat-lib:SW_Push_MP
- Y1: value 32MHz -> 32MHz 12pF; footprint (none) -> Crystal:Crystal_SMD_2016-4Pin_2.0x1.6mm; LCSC Part # (none) -> C2682773
- Y2: value 32.768kHz -> 32.768kHz 12.5pF; LCSC Part # (none) -> C5213671
Connections:
- net D+: now also J3.A6 (D+), J3.B6 (D+)
- net D-: now also J3.A7 (D-), J3.B7 (D-)
- net GND: now also SW1.MP, SW10.MP, SW11.MP, SW12.MP, SW13.MP, SW14.MP, SW15.MP, SW16.MP, SW17.MP, SW18.MP, SW19.MP, SW2.MP, SW20.MP, SW21.MP, SW22.MP, SW23.MP, SW24.MP, SW25.MP, SW26.MP, SW27.MP, SW28.MP, SW29.MP, SW3.MP, SW30.MP, SW4.MP, SW5.MP, SW6.MP, SW7.MP, SW8.MP, SW9.MP, C21.2, C22.2, J2.2 (Pin_2), J3.A1 (GND), J3.A12 (GND), J3.B1 (GND), J3.B12 (GND), J3.S1 (SHIELD), JP1.1 (A), Q2.2 (S), R10.1, R11.2, R12.2, R4.1, R5.1, R6.1, SW31.3 (C), U2.17 (VSS), U2.4 (~{CE}), U2.5 (EN2), U2.8 (VSS)
- net VBUS: now also C22.1, J3.A4 (VBUS), J3.A9 (VBUS), J3.B4 (VBUS), J3.B9 (VBUS), U2.13 (IN)
- net VDD_nRF: now also R3.1
- net ~{RESET}: now reaches U1.AC13 (P0.18/~{RESET})
- net ~{RESET}: now also U1.AD12 (P0.17), JP1.2 (B), R3.2
- new net: Q2.1 (G), R6.2, R7.1
- new net: J3.A5 (CC1), R11.1
- new net: J3.B5 (CC2), R12.1
- new net: D31.1 (K), R9.2
- new net: R10.2, U2.1 (TS)
- new net: R5.2, U2.12 (ILIM)
- new net: R4.2, U2.16 (ISET)
- new net: R9.1, U2.9 (~{CHG})
- new net: R8.1, SW31.1 (A)
- new net +5V: D31.2 (A), R7.2, U2.10 (OUT), U2.11 (OUT), U2.6 (EN1)
- new net +BATT: C21.1, J2.1 (Pin_1), R8.2, U2.2 (BAT), U2.3 (BAT)
- new net SYSOFF: Q2.3 (D), SW31.2 (B), U2.15 (SYSOFF)
- no-connect marks 1 -> 3
Other:
- note added: "3.3V"
- moved on the sheet: C14, C15, C16, C17, C18, C19, C20, C3, C4, D1, D10, D11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

Commit message: 2 Layers
Parts:
- removed D1, D10, D11, D12, D13, D14, D15, D16, D17, D18, D19, D2, D20, D21, D22, D23, D24, D25, D26, D27, D28, D29, D3, D30, D4, D5, D6, D7, D8, D9: D, symbol Device:D
- added D1, D10, D11, D12, D13, D14, D15, D16, D17, D18, D19, D2, D20, D21, D22, D23, D24, D25, D26, D27, D28, D29, D3, D32, D4, D5, D6, D7, D8, D9: 1N4148W, Diode_SMD:D_SOD-123, symbol Diode:1N4148W
- added R13: 10k, Resistor_SMD:R_0402_1005Metric_Pad0.72x0.64mm_HandSolder, symbol Device:R
- added SW32: SW_SPDT, ultraflat:Switch_Sink_MINI_MSK12CO2, symbol Switch:SW_SPDT
- C1, C2, C3, C4: LCSC Part # (none) -> C1548
- D31: footprint (none) -> LED_SMD:LED_0603_1608Metric_Pad1.05x0.95mm_HandSolder
- J1, J3: footprint Connector_USB:USB_C_Receptacle_HRO_TYPE-C-31-M-12 -> PCM_marbastlib-various:USB_C_Receptacle_HRO_TYPE-C-31-M-14
- SW31: footprint (none) -> ultraflat:Switch_Sink_MINI_MSK12CO2; LCSC Part # (none) -> C2681570
- U2: footprint Package_DFN_QFN:VQFN-16-1EP_3x3mm_P0.5mm_EP1.6x1.6mm -> Package_DFN_QFN:VQFN-16-1EP_3x3mm_P0.5mm_EP1.6x1.6mm_ThermalVias
Connections:
- net VDDH is gone; now on net +5V: C15.1, U1.Y2 (VDDH)
- net +BATT: now also R13.2
- net COL0: now also SW1.2, U1.J24 (NFC2/P0.10); no longer SW1.1
- net COL1: now also U1.A8 (AIN7/P0.31)
- net COL2: now also U1.A10 (AIN5/P0.29)
- net COL3: now also U1.A12 (AIN0/P0.02)
- net COL4: now also U1.A14 (P1.15)
- net COL5: now also U1.A16 (P1.13)
- net GND: now also SW32.3 (C)
- net ROW0: now also U1.A20 (P1.10), D1.1 (K), D2.1 (K), D3.1 (K), D32.1 (K), D4.1 (K), D5.1 (K)
- net ROW1: now also U1.Y23 (P1.01), D10.1 (K), D11.1 (K), D6.1 (K), D7.1 (K), D8.1 (K), D9.1 (K)
- net ROW2: now also U1.W24 (P1.02), D12.1 (K), D13.1 (K), D14.1 (K), D15.1 (K), D16.1 (K), D17.1 (K)
- net ROW3: now also U1.U24 (P1.04), D18.1 (K), D19.1 (K), D20.1 (K), D21.1 (K), D22.1 (K), D23.1 (K)
- net ROW4: now also U1.R24 (P1.06), D24.1 (K), D25.1 (K), D26.1 (K), D27.1 (K), D28.1 (K), D29.1 (K)
- net SYSOFF: now also SW32.2 (B)
- net at SW27.2: now also D26.2 (A)
- net at SW6.2: now also D5.2 (A)
- net at SW21.2: now also D20.2 (A)
- net at SW26.2: now also D25.2 (A)
- net at SW24.2: now also D23.2 (A)
- net at SW10.2: now also D9.2 (A)
- net DECUSB: now reaches C13.2, U1.AC5 (DECUSB)
- net DEC4_6: now reaches C11.2, C12.2, L3.2, U1.B5 (DEC4), U1.E24 (DEC6)
- net DEC1: now reaches C8.2, U1.C1 (DEC1)
- net DEC3: now reaches C9.2, U1.D23 (DEC3)
- net DEC5: now reaches C10.2, U1.N24 (DEC5)
- net at SW11.2: now also D10.2 (A)
- net at SW20.2: now also D19.2 (A)
- net at SW13.2: now also D12.2 (A)
- net at SW28.2: now also D27.2 (A)
- net at SW29.2: now also D28.2 (A)
- net at SW23.2: now also D22.2 (A)
- net at SW18.2: now also D17.2 (A)
- net at SW15.2: now also D14.2 (A)
- net at SW14.2: now also D13.2 (A)
- net at SW3.2: now also D2.2 (A)
- net at SW12.2: now also D11.2 (A)
- net at SW17.2: now also D16.2 (A)
- net at SW4.2: now also D3.2 (A)
- net at SW16.2: now also D15.2 (A)
- net at SW7.2: now also D6.2 (A)
- net at SW9.2: now also D8.2 (A)
- net at SW22.2: now also D21.2 (A)
- net at SW2.2: now also D1.2 (A)
- net at SW5.2: now also D4.2 (A)
- net at SW19.2: now also D18.2 (A)
- net at SW8.2: now also D7.2 (A)
- net at SW25.2: now also D24.2 (A)
- net at SW30.2: now also D29.2 (A)
- new net: D32.2 (A), SW1.1
- new net: R13.1, SW32.1 (A)
- no-connect marks 3 -> 38
Other:
- note added: "LS"
- moved on the sheet: AE1, C1, C10, C11, C12, C13, C2, C21, C22, C3, C4, C5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

Commit message: Case
Parts:
- added TP1, TP2, TP3, TP4: TestPoint, TestPoint:TestPoint_Pad_D1.5mm, symbol Connector:TestPoint
- C11, C17: LCSC Part # (none) -> C15849
- C13, C14, C15, C16, C21, C22: LCSC Part # (none) -> C19666
- C18, C19, C20, C8: LCSC Part # (none) -> C1525
- C9: LCSC Part # (none) -> C1546
- D31: LCSC Part # (none) -> C2290
- J1, J3: LCSC Part # C165948 -> C223907
- L2, L4: LCSC Part # (none) -> C1035
- Q2: LCSC Part # (none) -> C8545
- R1, R11, R12, R2: LCSC Part # (none) -> C25905
- R10, R13, R3, R6, R8: LCSC Part # (none) -> C25744
- R5, R9: LCSC Part # (none) -> C25867
- R7: LCSC Part # (none) -> C25076
- U1: LCSC Part # (none) -> C190794
Connections:
- net GND: now also TP4.1
- net VBUS: now also TP3.1
- net at U1.AA24 (SWDCLK): now also TP1.1
- net at U1.AC24 (SWDIO): now also TP2.1
- no-connect marks 38 -> 36
