File: hardware/left/leptosis-left.kicad_pcb (KiCad board)
At the start: 4 copper layers, 93.5 x 72.3 mm, 91 parts, among them J1 USB_C_Receptacle_USB2.0_14P, J2 Conn_01x02, Q2 2N7002, SW10 SW_Push, SW11 SW_Push, SW12 SW_Push, SW14 SW_Push, SW15 SW_Push, SW16 SW_Push, SW17 SW_Push, SW18 SW_Push, SW2 SW_Push, SW22 SW_Push, SW23 SW_Push, SW24 SW_Push, SW3 SW_Push, SW31 SW_SPDT, SW4 SW_Push, SW5 SW_Push, SW6 SW_Push, SW8 SW_Push, SW9 SW_Push, U1 nRF52840, U2 BQ24075RGT, U3 MAX17048X, Y1 32MHz 12pF, Y2 32.768kHz 12.5pF

Commit message: Finished!
Routing:
- net +BATT: track 63.3 -> 64.2 mm
- net GND: vias 140 -> 147
Changed lines of the file:
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@@
 	)
 	(paper "A4")
+	(title_block
+		(title "Leptosis")
+		(date "2025-07-06")
+		(rev "v1.1")
+		(company "Chengyin Yao (cheyao)")
+		(comment 1 "A PG1316 Split Keyboard")
+		(comment 2 "Solderpad License")
+	)
 	(layers
 		(0 "F.Cu" signal)
@@
 			)
 		)
-		(property "LCSC Part #" "C1035 "
+		(property "LCSC Part #" "C86083"
 			(at 0 0 180)
 			(unlocked yes)
@@
 			)
 		)
-		(property "LCSC Part #" "C1035 "
+		(property "LCSC Part #" "C86083"
 			(at 0 0 180)
 			(unlocked yes)
@@
 	)
 	(via
+		(at 128.82 99.94)
+		(size 0.6)
+		(drill 0.3)
+		(layers "F.Cu" "B.Cu")
+		(free yes)
+		(net 54)
+	)
+	(via
 		(at 149.61 110.48)
 		(size 0.6)
@@
 	)
 	(via
+		(at 122.59 86.24)
+		(size 0.6)
+		(drill 0.3)
+		(layers "F.Cu" "B.Cu")
+		(free yes)
+		(net 54)
+	)
+	(via
 		(at 168.870097 97.369104)
 		(size 0.6)
@@
 	)
 	(via
-		(at 160.370097 89.619104)
+		(at 130.98 91.52)
+		(size 0.6)
+		(drill 0.3)
+		(layers "F.Cu" "B.Cu")
+		(free yes)
+		(net 54)
+	)
+	(via
+		(at 162.027737 89.452263)
 		(size 0.6)
 		(drill 0.3)
@@
 	)
 	(via
+		(at 130.99 79.43)
+		(size 0.6)
+		(drill 0.3)
+		(layers "F.Cu" "B.Cu")
+		(free yes)
+		(net 54)
+	)
+	(via
 		(at 177.995097 94.019104)
 		(size 0.6)
@@
 	)
 	(via
+		(at 125.98 77.87)
+		(size 0.6)
+		(drill 0.3)
+		(layers "F.Cu" "B.Cu")
+		(free yes)
+		(net 54)
+	)
+	(via
 		(at 174.26 105.369104)
 		(size 0.6)
@@
 	)
 	(via
+		(at 133.33 94.13)
+		(size 0.6)
+		(drill 0.3)
+		(layers "F.Cu" "B.Cu")
+		(free yes)
+		(net 54)
+	)
+	(via
 		(at 167.120097 71.369104)
 		(size 0.6)
@@
 	)
 	(via
+		(at 164.76 85.83)
+		(size 0.6)
+		(drill 0.3)
+		(layers "F.Cu" "B.Cu")
+		(free yes)
+		(net 54)
+	)
+	(via
 		(at 179.370097 85.119104)
 		(size 0.6)
@@
 	(segment
 		(start 179.795097 93.139104)
+		(end 179.4 93.139104)
+		(width 0.5977)
+		(layer "B.Cu")
+		(net 55)
+	)
+	(segment
+		(start 179.4 93.139104)
 		(end 177.165097 93.139104)
 		(width 0.5977)
@@
 	)
 	(segment
-		(start 165.070097 87.069104)
-		(end 164.657597 87.069104)
-		(width 0.25)
-		(layer "B.Cu")
-		(net 65)
-	)
-	(segment
 		(start 167.580097 89.854104)
 		(end 167.180097 89.854104)
@@
 	)
 	(segment
+		(start 139.470097 108.73)
+		(end 139.470097 108.869104)
+		(width 0.5)
+		(layer "B.Cu")
+		(net 72)
+	)
+	(segment
+		(start 139.470097 108.869104)
+		(end 139.020097 109.319104)
+		(width 0.5)
+		(layer "B.Cu")
+		(net 72)
+	)
+	(segment
 		(start 136.220097 109.994104)
 		(end 135.520097 110.694104)
@@
 	(segment
 		(start 139.470097 108.449104)
-		(end 139.470097 108.869104)
-		(width 0.2)
-		(layer "B.Cu")
-		(net 72)
-	)
-	(segment
-		(start 139.470097 108.869104)
-		(end 139.920097 109.319104)
+		(end 139.470097 108.73)
 		(width 0.2)
 		(layer "B.Cu")
@@
 	)
 	(segment
+		(start 139.470097 108.869104)
+		(end 139.920097 109.319104)
+		(width 0.5)
+		(layer "B.Cu")
+		(net 72)
+	)
+	(segment
 		(start 135.520097 109.319104)
 		(end 135.520097 108.669104)
@@
 	)
 	(segment
-		(start 139.470097 108.869104)
-		(end 139.020097 109.319104)
-		(width 0.2)
+		(start 139.470097 108.449104)
+		(end 139.470097 109.319104)
+		(width 0.5)
 		(layer "B.Cu")
 		(net 72)
@@
 			)
 		)
+	)
+	(zone
+		(net 0)
+		(net_name "")
+		(layer "B.Cu")
+		(hatch edge 0.5)
+		(connect_pads
+			(clearance 0)
+		)
+		(min_thickness 0.25)
+		(filled_areas_thickness no)
+		(keepout
+			(tracks allowed)
+			(vias allowed)
+			(pads allowed)
+			(copperpour not_allowed)
+			(footprints allowed)
+		)
+		(placement
+			(enabled no)
+			(sheetname "/")
+		)
+		(fill
+			(thermal_gap 0.5)
+			(thermal_bridge_width 0.5)
+		)
+		(polygon
+			(pts
+				(xy 175.02 92.7) (xy 175.02 92.28) (xy 174.97 92.28) (xy 174.97 92.7)
+			)
+		)

Commit message: Finish
Connections:
- R7 pad 2: +5V -> VBUS
Routing:
- net +5V: track 12.0 -> 8.74 mm
- net VBUS: track 8.29 -> 11.1 mm
Other:
- board text removed: "301540 battery or 302025"
