File: hardware/right/leptosis-right.kicad_pcb (KiCad board)
At the start: 4 copper layers, 93.5 x 72.3 mm, 91 parts, among them J1 USB_C_Receptacle_USB2.0_14P, J2 Conn_01x02, Q2 2N7002, SW10 SW_Push, SW11 SW_Push, SW12 SW_Push, SW14 SW_Push, SW15 SW_Push, SW16 SW_Push, SW17 SW_Push, SW18 SW_Push, SW2 SW_Push, SW22 SW_Push, SW23 SW_Push, SW24 SW_Push, SW3 SW_Push, SW31 SW_SPDT, SW4 SW_Push, SW5 SW_Push, SW6 SW_Push, SW8 SW_Push, SW9 SW_Push, U1 nRF52840, U2 BQ24075RGT, U3 MAX17048X, Y1 32MHz 12pF, Y2 32.768kHz 12.5pF

Commit message: Finished!
Routing:
- net GND: vias 105 -> 110
Changed lines of the file:
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@@
 			)
 		)
-		(property "LCSC Part #" "C1035 "
+		(property "LCSC Part #" "C86083"
 			(at 0 0 0)
 			(unlocked yes)
@@
 			)
 		)
-		(property "LCSC Part #" "C1035 "
+		(property "LCSC Part #" "C86083"
 			(at 0 0 0)
 			(unlocked yes)
@@
 			(at 0 2.83 270)
 			(layer "B.SilkS")
+			(hide yes)
 			(effects
 				(font
@@
 	)
 	(gr_rect
-		(start 145.775001 120.324416)
-		(end 185.775001 135.324416)
+		(start 146.7 120.07)
+		(end 186.7 134.57)
 		(stroke
 			(width 0.1)
@@
 	)
 	(gr_text "+"
-		(at 130.975001 82.024416 0)
+		(at 146 114.75 180)
 		(layer "F.SilkS")
 		(effects
@@
 			)
 		)
-		(render_cache "+" 0
+		(render_cache "+" 180
 			(polygon
 				(pts
-					(xy 131.073004 81.454308) (xy 131.073004 81.88616) (xy 131.498444 81.88616) (xy 131.498444 82.062107)
-					(xy 131.073004 82.062107) (xy 131.073004 82.490753) (xy 130.879747 82.490753) (xy 130.879747 82.062107)
-					(xy 130.458702 82.062107) (xy 130.458702 81.88616) (xy 130.879747 81.88616) (xy 130.879747 81.454308)
+					(xy 145.901996 115.320107) (xy 145.901996 114.888255) (xy 145.476556 114.888255) (xy 145.476556 114.712308)
+					(xy 145.901996 114.712308) (xy 145.901996 114.283662) (xy 146.095253 114.283662) (xy 146.095253 114.712308)
+					(xy 146.516298 114.712308) (xy 146.516298 114.888255) (xy 146.095253 114.888255) (xy 146.095253 115.320107)
 				)
 			)
@@
 	)
 	(gr_text "-"
-		(at 138.075001 81.974416 0)
+		(at 138.9 114.8 180)
 		(layer "F.SilkS")
 		(effects
@@
 			)
 		)
-		(render_cache "-" 0
+		(render_cache "-" 180
 			(polygon
 				(pts
-					(xy 137.638387 82.01) (xy 137.638387 81.829657) (xy 138.518668 81.829657) (xy 138.518668 82.01)
+					(xy 139.336613 114.764415) (xy 139.336613 114.944758) (xy 138.456332 114.944758) (xy 138.456332 114.764415)
 				)
 			)
@@
 	)
 	(via
+		(at 112.273482 93.585663)
+		(size 0.6)
+		(drill 0.3)
+		(layers "F.Cu" "B.Cu")
+		(free yes)
+		(net 54)
+	)
+	(via
 		(at 112.53 99.274416)
 		(size 0.6)
@@
 	)
 	(via
+		(at 104.5 94.5)
+		(size 0.6)
+		(drill 0.3)
+		(layers "F.Cu" "B.Cu")
+		(free yes)
+		(net 54)
+	)
+	(via
 		(at 136.3 112.5)
 		(size 0.6)
@@
 	)
 	(via
+		(at 118.97 132.78)
+		(size 0.6)
+		(drill 0.3)
+		(layers "F.Cu" "B.Cu")
+		(free yes)
+		(net 54)
+	)
+	(via
 		(at 103.05 117.974416)
 		(size 0.6)
@@
 	)
 	(via
+		(at 106.66 98.66)
+		(size 0.6)
+		(drill 0.3)
+		(layers "F.Cu" "B.Cu")
+		(free yes)
+		(net 54)
+	)
+	(via
 		(at 100.15 94.49)
 		(size 0.6)
@@
 	)
 	(via
+		(at 112.88 91.91)
+		(size 0.6)
+		(drill 0.3)
+		(layers "F.Cu" "B.Cu")
+		(free yes)
+		(net 54)
+	)
+	(via
 		(at 110.94 97.54)
 		(size 0.6)
@@
 	)
 	(segment
-		(start 112.17 108.02)
-		(end 111.164416 107.014416)
+		(start 177.9 109.099416)
+		(end 177.9 107.9)
 		(width 0.2)
 		(layer "F.Cu")
@@
 	)
 	(segment
-		(start 109.94 107.014416)
-		(end 109.9 106.974416)
+		(start 160.9 106.08)
+		(end 160.9 104.849416)
 		(width 0.2)
 		(layer "F.Cu")
@@
 	)
 	(segment
-		(start 177.9 109.099416)
-		(end 177.9 107.9)
+		(start 109.9 103.601526)
+		(end 108.025398 101.726924)
 		(width 0.2)
 		(layer "F.Cu")
@@
 	)
 	(segment
-		(start 111.164416 107.014416)
-		(end 109.94 107.014416)
+		(start 109.9 106.974416)
+		(end 109.9 103.601526)
 		(width 0.2)
 		(layer "F.Cu")
@@
 	)
 	(segment
-		(start 160.9 106.08)
-		(end 160.9 104.849416)
+		(start 111.164416 107.014416)
+		(end 109.94 107.014416)
 		(width 0.2)
 		(layer "F.Cu")
@@
 	)
 	(segment
-		(start 109.9 103.601526)
-		(end 108.025398 101.726924)
+		(start 111.945 107.795)
+		(end 111.164416 107.014416)
 		(width 0.2)
 		(layer "F.Cu")
@@
 	)
 	(segment
-		(start 109.9 106.974416)
-		(end 109.9 103.601526)
+		(start 109.94 107.014416)
+		(end 109.9 106.974416)
 		(width 0.2)
 		(layer "F.Cu")
@@
 	)
 	(via
-		(at 112.17 108.02)
+		(at 111.945 107.795)
 		(size 0.6)
 		(drill 0.3)
@@
 		(width 0.2)
 		(layer "B.Cu")
+		(net 90)
+	)
+	(segment
+		(start 111.945 107.795)
+		(end 112.17 108.02)
+		(width 0.2)
+		(layer "B.Cu")

Commit message: Finish
Connections:
- R7 pad 2: +5V -> VBUS
Routing:
- net VBUS: track 11.1 -> 12.5 mm
- net +5V: track 16.0 -> 15.2 mm
